File: minigame-pcb.kicad_sch (KiCad schematic)
At the start: 87 parts, among them IC1 HT16K33A-28SSOP, J1 USB_C_Receptacle_USB2.0_16P, U2 AMS1117-3.3, U3 W25Q128JVS

Commit message: e
Parts:
- added C10, C11, C12, C13, C14, C3, C4, C8, C9: 100nF, symbol Device:C_Small_US
- added C15, C16: 1uF, symbol Device:C_Small_US
- added U4: RP2040, Package_DFN_QFN:QFN-56-1EP_7x7mm_P0.4mm_EP3.2x3.2mm, symbol MCU_RaspberryPi:RP2040
Connections:
- net +3V3: now also C10.1, C11.1, C12.1, C13.1, C14.1, C15.2, C8.1, C9.1, U4.1 (IOVDD), U4.10 (IOVDD), U4.22 (IOVDD), U4.33 (IOVDD), U4.42 (IOVDD), U4.43 (ADC_AVDD), U4.44 (VREG_IN), U4.48 (USB_VDD), U4.49 (IOVDD)
- net GND: now also C10.2, C11.2, C12.2, C13.2, C14.2, C15.1, C16.1, C3.2, C4.2, C8.2, C9.2
- net -5V: now reaches J1.A4 (VBUS), J1.A9 (VBUS), J1.B4 (VBUS), J1.B9 (VBUS)
- net -5V: no longer C6.2, U2.3 (VI)
- net at J1.A6 (D+), J1.B6 (D+): now also U4.47 (USB_DP)
- net at J1.A7 (D-), J1.B7 (D-): now also U4.46 (USB_DM)
- new net +1V1: C16.2, C3.1, C4.1, U4.23 (DVDD), U4.45 (VREG_VOUT), U4.50 (DVDD)
- new net +5V: C6.2, U2.3 (VI)
Other:
- moved on the sheet: C5, C6, C7, J1, JP1, R11, R12, R13, U2, U3

Commit message: e
Parts:
- removed C2: C_Small_US, Capacitor_SMD:C_0603_1608Metric_Pad1.08x0.95mm_HandSolder, symbol Device:C_Small_US
- removed JP1: Jumper_2_Small_Open, Jumper:Jumper_Harwin_S1621_P10.9mm, symbol Jumper:Jumper_2_Small_Open
- removed R12, R13: R_US, Resistor_SMD:R_0603_1608Metric_Pad0.98x0.95mm_HandSolder, symbol Device:R_US
- added C17, C18: 15pF, Capacitor_SMD:C_0603_1608Metric_Pad1.08x0.95mm_HandSolder, symbol Device:C_Small
- added JP2: Jumper_2_Small_Open, Jumper:Jumper_Harwin_S1621_P10.9mm, symbol Jumper:Jumper_2_Small_Open
- added R14, R17: 1K, Resistor_SMD:R_0603_1608Metric_Pad0.98x0.95mm_HandSolder, symbol Device:R_US
- added R15, R16: 27.4, Resistor_SMD:R_0603_1608Metric_Pad0.98x0.95mm_HandSolder, symbol Device:R_US
- added Y1: ABM8-272-T3, custom-project:XTAL_ABM8-272-T3, symbol Device:Crystal_GND24
- C1: value C_Small_US -> 0.1uF; footprint Capacitor_SMD:C_0603_1608Metric_Pad1.08x0.95mm_HandSolder -> (none)
- C5, C6: value C_Small_US -> 10u
- C7: value C_Small_US -> 100nF
- R1, R2: value R_US -> 4.7K
- R11: value R_US -> 5.1k
Connections:
- net -3V3 is gone; now on net +3V3: C5.2, U2.2 (VO)
- net +3V3: no longer C1.1
- net GND: now also U4.57 (GND), C17.1, C18.1, JP2.1 (A), Y1.2, Y1.4
- net at IC1.1 (VSS): no longer C1.2
- net at U4.20 (XIN): now also C17.2, Y1.1
- net at U4.21 (XOUT): now also R14.2
- net at U4.26 (RUN): now also C1.2
- net at J1.A7 (D-), J1.B7 (D-): now also R16.1; no longer U4.46 (USB_DM)
- net at J1.A6 (D+), J1.B6 (D+): now also R15.1; no longer U4.47 (USB_DP)
- net at U4.56 (QSPI_SS): now also R17.1
- net -5V renamed VBUS
- new net: C18.2, R14.1, Y1.3
- new net: JP2.2 (B), R17.2
- new net: R16.2, U4.46 (USB_DM)
- new net: R15.2, U4.47 (USB_DP)
- no-connect marks 0 -> 10
Other:
- moved on the sheet: C7, J1, R11

Commit message: e
Parts:
- removed D10, D11, D12, D13, D14, D15, D16, D17, D18, D19, D2, D20, D21, D22, D23, D24, D25, D26, D27, D28, D29, D3, D30, D31, D32, D33, D34, D35, D36, D37, D38, D39, D4, D40, D41, D42, D43, D44, D45, D46, D47, D48, D49, D5, D50, D51, D52, D53, D54, D55, D56, D57, D58, D59, D6, D60, D61, D62, D63, D64, D7, D8, D9: LED, LED_SMD:LED_0603_1608Metric_Pad1.05x0.95mm_HandSolder, symbol Device:LED
- removed IC1: HT16K33A-28SSOP, HT16K33A:SOP64P600X175-28N, symbol HT16K33A:HT16K33A-28SSOP
- removed R10, R3, R4, R5, R6, R7, R8, R9: R_US, symbol Device:R_US
- removed R2: 4.7K, Resistor_SMD:R_0603_1608Metric_Pad0.98x0.95mm_HandSolder, symbol Device:R_US
- added D2, D3: SS34, Diode_SMD:D_SMA, symbol Diode:SS34
- added SW1: SW_Push, symbol Switch:SW_Push
- R1: value 4.7K -> 10k
Connections:
- net +3V3: now also R1.2
- net +5V: now also D3.2 (A); no longer C6.2, U2.3 (VI)
- net GND: now also C1.1, D1.1 (K), SW1.2
- net test-led: now reaches D1.2 (A)
- net test-led: now also U4.37 (GPIO25)
- net at R1.1: now also C1.2, U4.26 (RUN), SW1.1
- net qspi_ss: now reaches U3.1 (~{CS})
- net qspi_ss: now also R17.1, U4.56 (QSPI_SS)
- net qspi_sd1: now reaches U3.2 (DO/IO_{1})
- net qspi_sd1: now also U4.55 (QSPI_SD1)
- net qspi_sd2: now reaches U3.3 (~{WP}/IO_{2})
- net qspi_sd2: now also U4.54 (QSPI_SD2)
- net qspi_sd0: now reaches U3.5 (DI/IO_{0})
- net qspi_sd0: now also U4.53 (QSPI_SD0)
- net qspi_sclk: now reaches U3.6 (CLK)
- net qspi_sclk: now also U4.52 (QSPI_SCLK)
- net qspi_sd3: now reaches U3.7 (~{HOLD}/~{RESET}/IO_{3})
- net qspi_sd3: now also U4.51 (QSPI_SD3)
- net xout: now reaches C18.2, R14.1, Y1.3
- net xin: now reaches C17.2, U4.20 (XIN), Y1.1
- net D-: now reaches J1.A7 (D-), J1.B7 (D-), R16.1
- net D+: now reaches J1.A6 (D+), J1.B6 (D+), R15.1
- new net: C6.2, D2.1 (K), D3.1 (K), U2.3 (VI)
- new net +BATT: D2.2 (A)
- no-connect marks 10 -> 2
Other:
- moved on the sheet: C1, C17, C18, C5, C6, C7, R14, U2, U3, Y1
