File: _autosave-minigame-pcb.kicad_sch (KiCad schematic)
At the start: 88 parts, among them IC1 HT16K33A-28SSOP, J1 USB_C_Receptacle_USB2.0_16P, U1 RP2040, U2 AMS1117-3.3, U3 W25Q128JVS

Commit message: e
Parts:
- removed U1: RP2040, RP2040:QFN40P700X700X90-57N, symbol RP2040-new:RP2040
